Commit message: kauil gazebo

File: catkin_ws/src/Kauil_description/urdf/Kauil.xacro (robot description, xacro)
@@ -1,7 +1,7 @@
 <?xml version="1.0" ?>
-<robot name="KauilURDF" xmlns:xacro="http://www.ros.org/wiki/xacro">
-<xacro:include filename="$(find KauilURDF_description)/urdf/materials.xacro" />
-<xacro:include filename="$(find KauilURDF_description)/urdf/KauilURDF.trans" />
-<xacro:include filename="$(find KauilURDF_description)/urdf/KauilURDF.gazebo" />
+<robot name="Kauil" xmlns:xacro="http://www.ros.org/wiki/xacro">
+<xacro:include filename="$(find Kauil_description)/urdf/materials.xacro" />
+<xacro:include filename="$(find Kauil_description)/urdf/Kauil.trans" />
+<xacro:include filename="$(find Kauil_description)/urdf/Kauil.gazebo" />
 <link name="base_link">
   <inertial>
@@ -13,5 +13,5 @@
     <origin xyz="0 0 0" rpy="0 0 0"/>
     <geometry>
-      <mesh filename="package://KauilURDF_description/meshes/base_link.stl" scale="0.001 0.001 0.001"/>
+      <mesh filename="package://Kauil_description/meshes/base_link.stl" scale="0.001 0.001 0.001"/>
     </geometry>
     <material name="silver"/>
@@ -20,5 +20,5 @@
     <origin xyz="0 0 0" rpy="0 0 0"/>
     <geometry>
-      <mesh filename="package://KauilURDF_description/meshes/base_link.stl" scale="0.001 0.001 0.001"/>
+      <mesh filename="package://Kauil_description/meshes/base_link.stl" scale="0.001 0.001 0.001"/>
     </geometry>
   </collision>
@@ -33,5 +33,5 @@
     <origin xyz="0.00546 -0.37938 -0.23895" rpy="0 0 0"/>
     <geometry>
-      <mesh filename="package://KauilURDF_description/meshes/camera_kauil_1.stl" scale="0.001 0.001 0.001"/>
+      <mesh filename="package://Kauil_description/meshes/camera_kauil_1.stl" scale="0.001 0.001 0.001"/>
     </geometry>
     <material name="silver"/>
@@ -40,5 +40,5 @@
     <origin xyz="0.00546 -0.37938 -0.23895" rpy="0 0 0"/>
     <geometry>
-      <mesh filename="package://KauilURDF_description/meshes/camera_kauil_1.stl" scale="0.001 0.001 0.001"/>
+      <mesh filename="package://Kauil_description/meshes/camera_kauil_1.stl" scale="0.001 0.001 0.001"/>
     </geometry>
   </collision>
@@ -53,5 +53,5 @@
     <origin xyz="-0.000825 -0.351848 -0.35095" rpy="0 0 0"/>
     <geometry>
-      <mesh filename="package://KauilURDF_description/meshes/hokuyo_kauil_1.stl" scale="0.001 0.001 0.001"/>
+      <mesh filename="package://Kauil_description/meshes/hokuyo_kauil_1.stl" scale="0.001 0.001 0.001"/>
     </geometry>
     <material name="silver"/>
@@ -60,5 +60,5 @@
     <origin xyz="-0.000825 -0.351848 -0.35095" rpy="0 0 0"/>
     <geometry>
-      <mesh filename="package://KauilURDF_description/meshes/hokuyo_kauil_1.stl" scale="0.001 0.001 0.001"/>
+      <mesh filename="package://Kauil_description/meshes/hokuyo_kauil_1.stl" scale="0.001 0.001 0.001"/>
     </geometry>
   </collision>
@@ -73,5 +73,5 @@
     <origin xyz="-0.26 -0.040001 -0.038107" rpy="0 0 0"/>
     <geometry>
-      <mesh filename="package://KauilURDF_description/meshes/r_wheel_1.stl" scale="0.001 0.001 0.001"/>
+      <mesh filename="package://Kauil_description/meshes/r_wheel_1.stl" scale="0.001 0.001 0.001"/>
     </geometry>
   </collision>
@@ -86,5 +86,5 @@
     <origin xyz="0.26 -0.040001 -0.038107" rpy="0 0 0"/>
     <geometry>
-      <mesh filename="package://KauilURDF_description/meshes/l_wheel_1.stl" scale="0.001 0.001 0.001"/>
+      <mesh filename="package://Kauil_description/meshes/l_wheel_1.stl" scale="0.001 0.001 0.001"/>
     </geometry>
   </collision>
@@ -170,5 +170,5 @@
     </ray>
     <plugin name="gazebo_ros_head_hokuyo_controller" filename="libgazebo_ros_gpu_laser.so">
-      <topicName>/kauil/laser/scan</topicName>
+      <topicName>/Kauil/laser/scan</topicName>
       <frameName>hokuyo_link</frameName>
     </plugin>
@@ -203,5 +203,5 @@
       <alwaysOn>true</alwaysOn>
       <updateRate>0.0</updateRate>
-      <cameraName>kauil/camera1</cameraName>
+      <cameraName>Kauil/camera1</cameraName>
       <imageTopicName>image_raw</imageTopicName>
       <cameraInfoTopicName>camera_info</cameraInfoTopicName>

File: catkin_ws/src/Kauil_description/urdf/materials.xacro (robot description, xacro)
@@ -1,4 +1,4 @@
 <?xml version="1.0" ?>
-<robot name="KauilURDF" xmlns:xacro="http://www.ros.org/wiki/xacro" >
+<robot name="Kauil" xmlns:xacro="http://www.ros.org/wiki/xacro" >
 <material name="silver">
   <color rgba="0.700 0.700 0.700 1.000"/>
